File: AS5600 Breakout.sch (KiCad schematic (older format))
At the start: 9 parts, among them J1 Conn_01x07, U1 AS5600

Commit message: updated schematic symbols
Parts:
- C1: symbol AS5600-Breakout-rescue:C-AS5600-Breakout-rescue -> Device:C
- C2, C3: symbol AS5600-Breakout-rescue:C-AS5600-Breakout-rescue -> AS5600-Breakout-rescue:C-AS5600-Breakout-rescue-AS5600-Breakout-rescue
- J1: symbol AS5600-Breakout-rescue:Conn_01x07-AS5600-Breakout-rescue -> AS5600-Breakout-rescue:Conn_01x07-AS5600-Breakout-rescue-AS5600-Breakout-rescue
- R1, R2, R3, R4: symbol AS5600-Breakout-rescue:R-AS5600-Breakout-rescue -> Device:R
- U1: symbol AS5600-Breakout-rescue:AS5600-AS5600-Breakout-rescue -> AS5600-Breakout-rescue:AS5600-AS5600-Breakout-rescue-AS5600-Breakout-rescue
Changed lines of the file:
@@
 $EndDescr
 $Comp
-L AS5600-Breakout-rescue:AS5600-AS5600-Breakout-rescue U1
+L AS5600-Breakout-rescue:AS5600-AS5600-Breakout-rescue-AS5600-Breakout-rescue U1
 U 1 1 5B77739F
 P 5500 4300
@@
 $EndComp
 $Comp
-L AS5600-Breakout-rescue:C-AS5600-Breakout-rescue C2
+L AS5600-Breakout-rescue:C-AS5600-Breakout-rescue-AS5600-Breakout-rescue C2
 U 1 1 5B7775CB
 P 5050 3950
@@
 $EndComp
 $Comp
-L AS5600-Breakout-rescue:GND-AS5600-Breakout-rescue #PWR01
+L AS5600-Breakout-rescue:GND-AS5600-Breakout-rescue-AS5600-Breakout-rescue #PWR01
 U 1 1 5B777636
 P 5050 3750
@@
 $EndComp
 $Comp
-L AS5600-Breakout-rescue:GND-AS5600-Breakout-rescue #PWR02
+L AS5600-Breakout-rescue:GND-AS5600-Breakout-rescue-AS5600-Breakout-rescue #PWR02
 U 1 1 5B77765C
 P 6400 3100
@@
 	5000 4150 5050 4150
 $Comp
-L AS5600-Breakout-rescue:C-AS5600-Breakout-rescue C1
+L Device:C C1
 U 1 1 5B777736
 P 4700 4050
@@
 $EndComp
 $Comp
-L AS5600-Breakout-rescue:GND-AS5600-Breakout-rescue #PWR03
+L AS5600-Breakout-rescue:GND-AS5600-Breakout-rescue-AS5600-Breakout-rescue #PWR03
 U 1 1 5B77776C
 P 4700 3850
@@
 $EndComp
 $Comp
-L AS5600-Breakout-rescue:GND-AS5600-Breakout-rescue #PWR04
+L AS5600-Breakout-rescue:GND-AS5600-Breakout-rescue-AS5600-Breakout-rescue #PWR04
 U 1 1 5B77778C
 P 5050 4500
@@
 	6900 2950 6900 3000
 Wire Wire Line
-	6150 4150 6200 4150
-Wire Wire Line
 	6150 4250 6550 4250
 Wire Wire Line
@@
 	6150 4450 6250 4450
 $Comp
-L AS5600-Breakout-rescue:R-AS5600-Breakout-rescue R1
+L Device:R R1
 U 1 1 5B777C09
 P 6700 4100
@@
 $EndComp
 $Comp
-L AS5600-Breakout-rescue:R-AS5600-Breakout-rescue R2
+L Device:R R2
 U 1 1 5B777C78
 P 6700 4500
@@
 Connection ~ 6550 4350
 $Comp
-L AS5600-Breakout-rescue:Conn_01x07-AS5600-Breakout-rescue J1
+L AS5600-Breakout-rescue:Conn_01x07-AS5600-Breakout-rescue-AS5600-Breakout-rescue J1
 U 1 1 5B78A669
 P 6600 2750
@@
 5V
 $Comp
-L AS5600-Breakout-rescue:R-AS5600-Breakout-rescue R3
+L Device:R R3
 U 1 1 5C26F27D
 P 6200 4000
@@
 $EndComp
 $Comp
-L AS5600-Breakout-rescue:GND-AS5600-Breakout-rescue #PWR05
+L AS5600-Breakout-rescue:GND-AS5600-Breakout-rescue-AS5600-Breakout-rescue #PWR05
 U 1 1 5C26F2B4
 P 6200 3800
@@
 Wire Wire Line
 	6200 3800 6200 3850
-Connection ~ 6200 4150
 Text GLabel 6300 3000 3    45   Input ~ 0
 VIN
 $Comp
-L AS5600-Breakout-rescue:C-AS5600-Breakout-rescue C3
+L AS5600-Breakout-rescue:C-AS5600-Breakout-rescue-AS5600-Breakout-rescue C3
 U 1 1 5C26F570
 P 5300 2850
@@
 $EndComp
 $Comp
-L AS5600-Breakout-rescue:R-AS5600-Breakout-rescue R4
+L Device:R R4
 U 1 1 5C26F640
 P 5050 2700
@@
 $EndComp
 $Comp
-L AS5600-Breakout-rescue:GND-AS5600-Breakout-rescue #PWR06
+L AS5600-Breakout-rescue:GND-AS5600-Breakout-rescue-AS5600-Breakout-rescue #PWR06
 U 1 1 5C26F707
 P 5300 3050
@@
 	6550 4350 6150 4350
 Wire Wire Line
+	5300 2700 5650 2700
+Wire Wire Line
+	6550 4350 6550 4500
+Wire Wire Line
+	6550 4100 6550 4250
+Wire Wire Line
+	6850 4100 7050 4100
+Wire Wire Line
+	6850 4500 7050 4500
+Wire Wire Line
+	7050 4100 7050 4500
+Connection ~ 6200 4150
+Wire Wire Line
 	6200 4150 6250 4150
 Wire Wire Line
-	5300 2700 5650 2700
-Wire Wire Line
-	6550 4350 6550 4500
-Wire Wire Line
-	6550 4100 6550 4250
-Wire Wire Line
-	6850 4100 7050 4100
-Wire Wire Line
-	6850 4500 7050 4500
-Wire Wire Line
-	7050 4100 7050 4500
+	6150 4150 6200 4150
 $EndSCHEMATC

Commit message: updating symbols
Parts:
- C2, C3: symbol AS5600-Breakout-rescue:C-AS5600-Breakout-rescue-AS5600-Breakout-rescue -> Device:C
- J1: symbol AS5600-Breakout-rescue:Conn_01x07-AS5600-Breakout-rescue-AS5600-Breakout-rescue -> Connector:Conn_01x07_Male
- U1: symbol AS5600-Breakout-rescue:AS5600-AS5600-Breakout-rescue-AS5600-Breakout-rescue -> AS5600:AS5600
Connections:
- wire segments 35 -> 34
Changed lines of the file:
@@
 $EndDescr
 $Comp
-L AS5600-Breakout-rescue:AS5600-AS5600-Breakout-rescue-AS5600-Breakout-rescue U1
+L AS5600:AS5600 U1
 U 1 1 5B77739F
 P 5500 4300
@@
 $EndComp
 $Comp
-L AS5600-Breakout-rescue:C-AS5600-Breakout-rescue-AS5600-Breakout-rescue C2
+L Device:C C2
 U 1 1 5B7775CB
 P 5050 3950
@@
 $EndComp
 $Comp
-L AS5600-Breakout-rescue:GND-AS5600-Breakout-rescue-AS5600-Breakout-rescue #PWR01
+L power:GND #PWR01
 U 1 1 5B777636
 P 5050 3750
@@
 $EndComp
 $Comp
-L AS5600-Breakout-rescue:GND-AS5600-Breakout-rescue-AS5600-Breakout-rescue #PWR02
+L power:GND #PWR02
 U 1 1 5B77765C
 P 6400 3100
@@
 $EndComp
 $Comp
-L AS5600-Breakout-rescue:GND-AS5600-Breakout-rescue-AS5600-Breakout-rescue #PWR03
+L power:GND #PWR03
 U 1 1 5B77776C
 P 4700 3850
@@
 $EndComp
 $Comp
-L AS5600-Breakout-rescue:GND-AS5600-Breakout-rescue-AS5600-Breakout-rescue #PWR04
+L power:GND #PWR04
 U 1 1 5B77778C
 P 5050 4500
@@
 Connection ~ 6550 4350
 $Comp
-L AS5600-Breakout-rescue:Conn_01x07-AS5600-Breakout-rescue-AS5600-Breakout-rescue J1
+L Connector:Conn_01x07_Male J1
 U 1 1 5B78A669
 P 6600 2750
@@
 F 3 "" H 6600 2750 50  0001 C CNN
 	1    6600 2750
-	0    1    -1   0
+	0    -1   1    0
 $EndComp
 Text GLabel 7050 4300 2    45   Input ~ 0
@@
 $EndComp
 $Comp
-L AS5600-Breakout-rescue:GND-AS5600-Breakout-rescue-AS5600-Breakout-rescue #PWR05
+L power:GND #PWR05
 U 1 1 5C26F2B4
 P 6200 3800
@@
 VIN
 $Comp
-L AS5600-Breakout-rescue:C-AS5600-Breakout-rescue-AS5600-Breakout-rescue C3
+L Device:C C3
 U 1 1 5C26F570
 P 5300 2850
@@
 $EndComp
 $Comp
-L AS5600-Breakout-rescue:GND-AS5600-Breakout-rescue-AS5600-Breakout-rescue #PWR06
+L power:GND #PWR06
 U 1 1 5C26F707
 P 5300 3050
@@
 	5300 3050 5300 3000
 Wire Wire Line
-	5200 2700 5300 2700
-Wire Wire Line
 	4900 2700 4850 2700
-Connection ~ 5300 2700
 Text GLabel 4850 2700 0    45   Input ~ 0
 VIN
@@
 	6550 4350 6150 4350
 Wire Wire Line
-	5300 2700 5650 2700
-Wire Wire Line
 	6550 4350 6550 4500
 Wire Wire Line
@@
 Wire Wire Line
 	6150 4150 6200 4150
+Wire Wire Line
+	5200 2700 5650 2700
 $EndSCHEMATC
